Commit message: Fix LIDAR orientation, map save order, and camera feed in RTT mode
- lidar.xacro: rotate laser_frame 180° (rpy="0 0 3.14159265") — LIDAR was
  physically mounted backwards, causing inverted SLAM maps
- phoenix_launcher.py: save SLAM map before killing processes so map_saver_cli
  can still subscribe to /map; fixes persistent "Map save failed" on RTT stop
- phoenix_launcher.py: start_raw_camera() / stop_raw_camera() — direct
  rpicam-vid MJPEG stream in manual and RTT modes (camera_detector only runs
  in autonomous mode)

Co-Authored-By: Claude Sonnet 4.6 <noreply@anthropic.com>

File: description/lidar.xacro (robot description, xacro)
@@ -4,5 +4,5 @@
         <parent link="chassis"/>
         <child link="laser_frame"/>
-        <origin xyz="0.122 0 0.212" rpy="0 0 0"/>
+        <origin xyz="0.122 0 0.212" rpy="0 0 3.14159265"/>
     </joint>
     <link name="laser_frame">
